File: hw/kicad/Reader.kicad_sch (KiCad schematic)
At the start: 61 parts, among them CN1 CN_1X3M, CN2 CN_USB-C, CN3 CN_1X2M, M1 MOD_RFID_NFC_PN532, Q1 TRS_NPN_123, Q2 TRS_NPN_123, Q3 TRS_NPN_123, Q4 TRS_NPN_123, SW1 Tact_Switch, SW2 Tact_Switch_2pin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

Commit message: Files updated
Connections:
- net at D6.2 (Dout): now also D7.4 (Din)
- net at D4.2 (Dout): now also D5.4 (Din)

Commit message: Fixes to make board suitable for local manucatruing
- Track made 0.2 min
- Pads 0.2 min(CP2102)
- Another bug fixes...
Connections:
- net at D6.2 (Dout): now also D7.4 (Din)
- net at D4.2 (Dout): now also D5.4 (Din)
Changed lines of the file:
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@@
 	)
 	(symbol
+		(lib_name "Reader-altium-import:root_0_DIO_LED_WS2812_5050")
 		(lib_id "Reader-altium-import:root_0_DIO_LED_WS2812_5050")
 		(at 457.5 184.989 0)
@@
 	)
 	(symbol
+		(lib_name "Reader-altium-import:root_0_DIO_LED_WS2812_5050")
 		(lib_id "Reader-altium-import:root_0_DIO_LED_WS2812_5050")
 		(at 377.5 184.989 0)
@@
 	)
 	(symbol
+		(lib_name "Reader-altium-import:root_0_DIO_LED_WS2812_5050")
 		(lib_id "Reader-altium-import:root_0_DIO_LED_WS2812_5050")
 		(at 417.5 184.989 0)
@@
 	)
 	(symbol
+		(lib_name "Reader-altium-import:root_0_DIO_LED_WS2812_5050")
 		(lib_id "Reader-altium-import:root_0_DIO_LED_WS2812_5050")
 		(at 497.5 184.989 0)
