File: hw/rev.1.0/PRISMO-reader.kicad_pcb (KiCad board)
At the start: 2 copper layers, 50 x 51 mm, 49 parts, among them J1 Conn_01x03, J3 PN532 Connector, J4 External 5V power, J5 USB4120-03-C_REVA, K1 G5LE-1, Q1 2N7002, Q2 BC847, Q3 BC847, SW1 Logout button, U1 ESP32-WROOM-32D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

Commit message: Bugfix with CP2102 connection (#15)
* fixed CP2102 peripheral connection

* renamed leds in order of connection
Parts:
- removed R4: 10k, Resistor_SMD:R_0805_2012Metric_Pad1.20x1.40mm_HandSolder
- R14: value 1k -> 10k
- turned R14 to 180 degrees
- renumbered D3 to D1, D4 to D2, D2 to D3, D1 to D4
Connections:
- R14 pad 1: Net-(U2-VIO) -> +5V
- U2 pad 15: Net-(U2-~{SUSPEND}) -> unconnected-(U2-~{SUSPEND}-Pad15)
- U2 pad 5: Net-(U2-VIO) -> unconnected-(U2-VIO-Pad5)
Routing:
- net Net-(U2-VIO): track 12.4 -> 0.00 mm, vias 2 -> 0
- net +5V: track 208.3 -> 218.1 mm
- net Net-(U2-~{SUSPEND}): track 8.84 -> 0.00 mm, vias 2 -> 0
- net GND: track 237.1 -> 235.2 mm
- net Net-(U2-~{RST}): track 7.82 -> 9.56 mm
- net Net-(U2-VDD): track 10.2 -> 8.94 mm
- net /UART_TX: track 28.2 -> 29.5 mm
